File: hardware/basic/kicad/yarrow_counter_basic.kicad_sch (KiCad schematic)
At the start: 58 parts, among them J1 USB-C, J2 SWD, J3 BOOT0, J4 TUBE (anode, cathode), Q1 600V N-MOSFET, Q2 2N7002, SW1 NRST, U1 CH32F203C8T6, U2 AP2112K-3.3, U3 USBLC6-2SC6, U4 TLV3201, U5 74AHCT1G04, Y1 8MHz

Commit message: Hardware: PCB placement of the Basic board with high-voltage rules, DRC baseline
Parts:
- removed J4: TUBE (anode, cathode), Connector_PinHeader_2.54mm:PinHeader_1x02_P2.54mm_Vertical, symbol Connector:Conn_01x02_Pin
- added J4: tube clip, anode, TestPoint:TestPoint_THTPad_D3.0mm_Drill1.5mm, symbol Connector:Conn_01x01_Pin
- added J5: tube clip, cathode, TestPoint:TestPoint_THTPad_D3.0mm_Drill1.5mm, symbol Connector:Conn_01x01_Pin
- C1, C2: footprint Capacitor_SMD:C_1206_3216Metric -> Capacitor_SMD:C_1812_4532Metric
- Q1: footprint Package_TO_SOT_SMD:SOT-223 -> Package_TO_SOT_SMD:TO-252-3_TabPin2
Connections:
- net ANODE: now also J4.1 (Pin_1)
- net GND: now also J5.1 (Pin_1)
